File: Flip/flip.kicad_pcb (KiCad board)
At the start: 2 copper layers, 95 x 62 mm, 18 parts, among them J1 CHANNEL, J2 COILS, J3 IDC1, J4 GROUND, J5 IDC2, Q1 Q_NPN_BEC, Q2 Q_NPN_BEC, Q3 Q_NPN_BEC, Q4 Q_NPN_BEC

Commit message: new PCB WIP
Parts:
- removed C1: 100nF, Capacitors_SMD:C_0805_HandSoldering
- removed TP1: HAL_TEST, Pin_Headers:Pin_Header_Straight_1x01_Pitch2.54mm
- added D1: D_COIL, Diodes_SMD:D_0805, F.Cu at (191.2, 114.6)
- added D2: D_COIL, Diodes_SMD:D_0805, F.Cu at (191.2, 133.8)
- added R5: [10k], Resistors_SMD:R_0603_HandSoldering, F.Cu at (181.7, 141.2)
- added R6: [10k], Resistors_SMD:R_0603_HandSoldering, F.Cu at (187.3, 143.9)
- J3: footprint Pin_Headers:Pin_Header_Straight_2x12_Pitch2.54mm -> #MOJABIBLIOTEKA:IDC_edge
- J5: value IDC2 -> HAL_TEST; footprint Pin_Headers:Pin_Header_Straight_2x12_Pitch2.54mm -> Pin_Headers:Pin_Header_Straight_1x03_Pitch2.54mm
- moved R1 43.2 mm to (250.0, 64.1)
- moved Q2 43.0 mm to (245.0, 69.3)
- moved Q3 43.0 mm to (249.0, 69.3)
- moved Q4 43.0 mm to (241.0, 69.3)
- moved R2 43.0 mm to (246.0, 64.4)
- moved R3 43.0 mm to (248.0, 64.4)
- moved R4 43.0 mm to (244.0, 64.4)
- moved Q1 42.8 mm to (254.0, 70.0)
- moved J5 34.5 mm to (190.6, 140.1)
- moved J3 32.1 mm to (236.0, 104.3)
- moved L1 25.1 mm to (191.1, 120.2)
- moved L2 21.4 mm to (191.2, 128.2)
- moved HG1 5.00 mm to (184.4, 140.1)
Connections:
- J3 pad 1: VCC -> GND
- J3 pad 2: GND -> VCC
- J3 pad 3: GND -> VCC
- J3 pad 4: VCC -> GND
- J4 pad 1: GND3 -> GND2
- J4 pad 3: GND2 -> GND3
- J5 pad 2: GND -> SW_GND
- J5 pad 3: GND -> DIGITAL
Routing:
- net Net-(D1-Pad2): track 107.1 -> 0.00 mm
- net Net-(D1-Pad1): track 101.2 -> 0.00 mm
- net DIGITAL: track 92.8 -> 0.00 mm
- net CH05: track 49.8 -> 0.00 mm
- net VCC: track 48.3 -> 0.00 mm, vias 1 -> 0
- net Net-(D2-Pad2): track 48.2 -> 0.00 mm, vias 1 -> 0
- net CH04: track 47.4 -> 0.00 mm
- net CH03: track 45.1 -> 0.00 mm
- net CH02: track 42.8 -> 0.00 mm
- net CH01: track 40.4 -> 0.00 mm
- net GND: track 35.2 -> 0.00 mm
- net CH16: track 54.5 -> 22.9 mm
- net CH15: track 56.9 -> 26.2 mm
- net GND0: track 44.8 -> 14.5 mm, vias 1 -> 0
- net CH14: track 59.1 -> 29.6 mm
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