File: kicad/flip.sch (KiCad schematic (older format))
At the start: 20 parts, among them J1 CHANNEL, J2 COILS, J3 IDC1, J4 GROUND, J5 HAL_TEST, Q1 Q_NPN_BEC, Q2 Q_NPN_BEC, Q3 Q_NPN_BEC, Q4 Q_NPN_BEC

Commit message: new PCB ready
Parts:
- removed J1: CHANNEL, Pin_Headers:Pin_Header_Straight_2x16_Pitch2.00mm, symbol CONN_02X16
- removed J4: GROUND, Pin_Headers:Pin_Header_Straight_2x04_Pitch2.00mm, symbol CONN_02X04
- added GND0: G4, #MOJABIBLIOTEKA:Jumper_SMD, symbol Jumper_NO_Small
- added GND1: G3, #MOJABIBLIOTEKA:Jumper_SMD, symbol Jumper_NO_Small
- added GND2: G1, #MOJABIBLIOTEKA:Jumper_SMD, symbol Jumper_NO_Small
- added GND3: G2, #MOJABIBLIOTEKA:Jumper_SMD, symbol Jumper_NO_Small
- added JP1: J1, #MOJABIBLIOTEKA:Jumper_SMD, symbol Jumper_NO_Small
- added JP10: J10, #MOJABIBLIOTEKA:Jumper_SMD, symbol Jumper_NO_Small
- added JP11: J11, #MOJABIBLIOTEKA:Jumper_SMD, symbol Jumper_NO_Small
- added JP12: J12, #MOJABIBLIOTEKA:Jumper_SMD, symbol Jumper_NO_Small
- added JP13: J13, #MOJABIBLIOTEKA:Jumper_SMD, symbol Jumper_NO_Small
- added JP14: J14, #MOJABIBLIOTEKA:Jumper_SMD, symbol Jumper_NO_Small
- added JP15: J15, #MOJABIBLIOTEKA:Jumper_SMD, symbol Jumper_NO_Small
- added JP16: J16, #MOJABIBLIOTEKA:Jumper_SMD, symbol Jumper_NO_Small
- added JP2: J2, #MOJABIBLIOTEKA:Jumper_SMD, symbol Jumper_NO_Small
- added JP3: J3, #MOJABIBLIOTEKA:Jumper_SMD, symbol Jumper_NO_Small
- added JP4: J4, #MOJABIBLIOTEKA:Jumper_SMD, symbol Jumper_NO_Small
- added JP5: J5, #MOJABIBLIOTEKA:Jumper_SMD, symbol Jumper_NO_Small
- added JP6: J6, #MOJABIBLIOTEKA:Jumper_SMD, symbol Jumper_NO_Small
- added JP7: J7, #MOJABIBLIOTEKA:Jumper_SMD, symbol Jumper_NO_Small
- added JP8: J8, #MOJABIBLIOTEKA:Jumper_SMD, symbol Jumper_NO_Small
- added JP9: J9, #MOJABIBLIOTEKA:Jumper_SMD, symbol Jumper_NO_Small
- J2: renamed from J3; footprint #MOJABIBLIOTEKA:IDC_edge -> Socket_Strips:Socket_Strip_Straight_2x12_Pitch2.54mm
- renumbered J5 to J1, J2 to J3, R5 to R2, R6 to R3, R2 to R4, R3 to R5, R4 to R6
Connections:
- net CH01: now also JP1.1
- net CH02: now also JP2.1
- net CH03: now also JP3.1
- net CH04: now also JP4.1
- net CH05: now also JP5.1
- net CH06: now also JP6.1
- net CH07: now also JP7.1
- net CH08: now also JP8.1
- net CH09: now also JP9.1
- net CH10: now also JP10.1
- net CH11: now also JP11.1
- net CH12: now also JP12.1
- net CH13: now also JP13.1
- net CH14: now also JP14.1
- net CH15: now also JP15.1
- net CH16: now also JP16.1
- net DIGITAL: now also JP1.2, JP10.2, JP11.2, JP12.2, JP13.2, JP14.2, JP15.2, JP16.2, JP2.2, JP3.2, JP4.2, JP5.2, JP6.2, JP7.2, JP8.2, JP9.2
- net GND0: now also GND0.1
- net GND1: now also GND1.1
- net GND2: now also GND2.1
- net GND3: now also GND3.1
- net SW_GND0: now also GND2.2
- net SW_GND1: now also GND3.2
- net SW_GND2: now also GND1.2
- net SW_GND3: now also GND0.2
Other:
- moved on the sheet: Q1, Q2, Q3, Q4, R1, R4, R5, R6
